Commit message: modify ankle

File: src/holosoma_retargeting/models/adam_sp/adam_sp_29dof_unuse.urdf (robot description, URDF)
Before this commit: robot adam_sp, 59 links, 58 joints
Links:
- added link heelPadLeft, mass 0.001; collision sphere radius=0.005; visual sphere radius=0.005
- added link heelPadRight, mass 0.001; collision sphere radius=0.005; visual sphere radius=0.005
- added link midfootPadLeftInner, mass 0.001; collision sphere radius=0.005; visual sphere radius=0.005
- added link midfootPadLeftOuter, mass 0.001; collision sphere radius=0.005; visual sphere radius=0.005
- added link midfootPadRightInner, mass 0.001; collision sphere radius=0.005; visual sphere radius=0.005
- added link midfootPadRightOuter, mass 0.001; collision sphere radius=0.005; visual sphere radius=0.005
- link toeLeftKeyframe: geometry 
- link toeRightKeyframe: geometry 
- link toeTipLeft: geometry collision sphere radius=0.005; visual sphere radius=0.005
- link toeTipRight: geometry collision sphere radius=0.005; visual sphere radius=0.005
Joints:
- added joint heelPad_Left: type fixed, parent toeLeft, child heelPadLeft, origin xyz=-0.075 0 -0.055 rpy=0 0 0
- added joint heelPad_Right: type fixed, parent toeRight, child heelPadRight, origin xyz=-0.075 0 -0.055 rpy=0 0 0
- added joint midfootPad_LeftInner: type fixed, parent toeLeft, child midfootPadLeftInner, origin xyz=0.05 -0.04 -0.055 rpy=0 0 0
- added joint midfootPad_LeftOuter: type fixed, parent toeLeft, child midfootPadLeftOuter, origin xyz=0.05 0.045 -0.055 rpy=0 0 0
- added joint midfootPad_RightInner: type fixed, parent toeRight, child midfootPadRightInner, origin xyz=0.05 0.04 -0.055 rpy=0 0 0
- added joint midfootPad_RightOuter: type fixed, parent toeRight, child midfootPadRightOuter, origin xyz=0.05 -0.045 -0.055 rpy=0 0 0
- joint toeTip_Left: origin xyz=0.14 0 -0.08 rpy=0 0 0 -> xyz=0.14 0 -0.05 rpy=0 0 0
- joint toeTip_Right: origin xyz=0.14 0 -0.08 rpy=0 0 0 -> xyz=0.14 0 -0.05 rpy=0 0 0
- joint toe_LeftKeyframe: origin xyz=0.0374996 0.0 -0.01 rpy=0 0 0 -> xyz=0.0 0.0 -0.01 rpy=0 0 0
- joint toe_RightKeyframe: origin xyz=0.0375023 0.0 -0.01 rpy=0 0 0 -> xyz=0.0 0.0 -0.01 rpy=0 0 0; parent toeRight -> anklePitchRight
