Commit message: fix(adam-pro): enable 29dof wrists in urdf for isaacsim

File: src/holosoma/holosoma/data/robots/adam_pro/adam_pro.urdf (robot description, URDF)
Before this commit: robot adam_pro, 57 links, 56 joints
Links:
- added link left_foot_contact_point, mass 0.001; visual box size=0.001 0.001 0.001
- added link right_foot_contact_point, mass 0.001; visual box size=0.001 0.001 0.001
Joints:
- added joint left_foot_contact_point: type fixed, parent toeLeft, child left_foot_contact_point, origin xyz=0 0 -0.037 rpy=0 0 0
- added joint right_foot_contact_point: type fixed, parent toeRight, child right_foot_contact_point, origin xyz=0 0 -0.037 rpy=0 0 0
- joint wristPitch_Left: axis (none) -> 0 1 0; limit (none) -> lower=-0.96 upper=0.96 effort=2.1 velocity=4.92; type fixed -> revolute
- joint wristPitch_Right: axis (none) -> 0 1 0; limit (none) -> lower=-0.96 upper=0.96 effort=2.1 velocity=4.92; type fixed -> revolute
- joint wristRoll_Left: axis (none) -> 1 0 0; limit (none) -> lower=-0.96 upper=0.96 effort=2.1 velocity=4.92; type fixed -> revolute
- joint wristRoll_Right: axis (none) -> 1 0 0; limit (none) -> lower=-0.96 upper=0.96 effort=2.1 velocity=4.92; type fixed -> revolute
- joint wristYaw_Left: axis (none) -> 0 0 1; limit (none) -> lower=-2.67 upper=2.67 effort=1.7 velocity=4.92; type fixed -> revolute
- joint wristYaw_Right: axis (none) -> 0 0 1; limit (none) -> lower=-2.67 upper=2.67 effort=1.7 velocity=4.92; type fixed -> revolute
